File: airbrake_mod.kicad_sch (KiCad schematic)
At the start: 9 parts

Commit message: Release Candidate 3
Fixed name, one location with vias. Added production files in prep for merge request.
Other:
- title: Airbrakes PCB - Earendel -> Airbrakes PCB - Veðrfölnir 
Changed lines of the file:
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@@
 	(paper "B")
 	(title_block
-		(title "Airbrakes PCB - Earendel")
+		(title "Airbrakes PCB - Veðrfölnir ")
 		(date "2025-02-18")
 		(rev "v2025.01A")
